File: minimix.kicad_sch (KiCad schematic)
At the start: 25 parts, among them J1 INOUT, J2 INOUT, J3 INOUT, J4 INOUT, J5 INOUT, J6 INOUT, J7 INOUT, J8 INOUT, SW1 SK23D05

Commit message: fixed typo
Other:
- company: Jan Marie Hemsing -> Jana Marie Hemsing
Changed lines of the file:
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@@
   (title_block
     (title "MINIMIX")
-    (date "2023-03-21")
-    (rev "v1.0.0")
-    (company "Jan Marie Hemsing")
+    (date "2023-03-26")
+    (rev "v1.0.1")
+    (company "Jana Marie Hemsing")
   )
   (junction (at 88.9 59.69) (diameter 0) (color 0 0 0 0)
